File: extras/KiCad/Basic_setup/Basic_Setup.kicad_sch (KiCad schematic)
At the start: 38 parts, among them J1 AUDIO, Y1 32.768kHz

Commit message: Doc
Parts:
- added R18: 270K, symbol Device:R
- added R19: 10M, symbol Device:R
Connections:
- net at C6.1, U1.10 (XO), Y1.1: now also R19.2
- net at C7.1, Y1.2: now also R18.1, R19.1; no longer U1.9 (XI)
- new net: R18.2, U1.9 (XI)
Other:
- moved on the sheet: C6, C7
Changed lines of the file:
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@@
 (kicad_sch (version 20230121) (generator eeschema)
-  (paper "User" 210.007 170.002)
+  (paper "User" 254 203.2)
   (title_block
     (title "BK1198 BASIC SETUP - VOLTAGE DIVIDER VERSION (SW BAND)")
@@
   (junction (at 146.05 107.95) (diameter 0) (color 0 0 0 0)
   )
-  (junction (at 114.3 109.22) (diameter 0) (color 0 0 0 0)
+  (junction (at 114.3 121.92) (diameter 0) (color 0 0 0 0)
   )
   (junction (at 158.75 72.39) (diameter 0) (color 0 0 0 0)
@@
   (junction (at 106.68 93.98) (diameter 0) (color 0 0 0 0)
   )
+  (junction (at 128.27 114.3) (diameter 0) (color 0 0 0 0)
+  )
   (junction (at 40.64 24.13) (diameter 0) (color 0 0 0 0)
   )
-  (junction (at 128.27 109.22) (diameter 0) (color 0 0 0 0)
+  (junction (at 128.27 121.92) (diameter 0) (color 0 0 0 0)
   )
   (junction (at 153.67 91.44) (diameter 0) (color 0 0 0 0)
@@
   (junction (at 156.21 99.06) (diameter 0) (color 0 0 0 0)
   )
-  (junction (at 121.92 116.84) (diameter 0) (color 0 0 0 0)
+  (junction (at 121.92 129.54) (diameter 0) (color 0 0 0 0)
   )
   (junction (at 86.36 24.13) (diameter 0) (color 0 0 0 0)
@@
   (junction (at 55.88 24.13) (diameter 0) (color 0 0 0 0)
   )
+  (junction (at 114.3 114.3) (diameter 0) (color 0 0 0 0)
+  )
   (junction (at 71.12 24.13) (diameter 0) (color 0 0 0 0)
   )
@@
     (stroke (width 0) (type default))
   )
+  (wire (pts (xy 125.73 114.3) (xy 128.27 114.3))
+    (stroke (width 0) (type default))
+  )
   (wire (pts (xy 158.75 72.39) (xy 158.75 78.74))
     (stroke (width 0) (type default))
@@
     (stroke (width 0) (type default))
   )
+  (wire (pts (xy 128.27 109.22) (xy 128.27 114.3))
+    (stroke (width 0) (type default))
+  )
   (wire (pts (xy 88.9 49.53) (xy 116.84 49.53))
     (stroke (width 0) (type default))
@@
     (stroke (width 0) (type default))
   )
-  (wire (pts (xy 114.3 116.84) (xy 121.92 116.84))
+  (wire (pts (xy 114.3 114.3) (xy 114.3 121.92))
+    (stroke (width 0) (type default))
+  )
+  (wire (pts (xy 114.3 129.54) (xy 121.92 129.54))
     (stroke (width 0) (type default))
   )
@@
     (stroke (width 0) (type default))
   )
-  (wire (pts (xy 128.27 97.79) (xy 128.27 109.22))
-    (stroke (width 0) (type default))
-  )
   (wire (pts (xy 95.25 93.98) (xy 106.68 93.98))
     (stroke (width 0) (type default))
@@
     (stroke (width 0) (type default))
   )
-  (wire (pts (xy 121.92 116.84) (xy 121.92 118.11))
+  (wire (pts (xy 121.92 129.54) (xy 121.92 130.81))
     (stroke (width 0) (type default))
   )
@@
     (stroke (width 0) (type default))
   )
+  (wire (pts (xy 118.11 114.3) (xy 114.3 114.3))
+    (stroke (width 0) (type default))
+  )
   (wire (pts (xy 69.85 83.82) (xy 80.01 83.82))
     (stroke (width 0) (type default))
@@
     (stroke (width 0) (type default))
   )
-  (wire (pts (xy 114.3 109.22) (xy 114.3 91.44))
+  (wire (pts (xy 114.3 91.44) (xy 114.3 114.3))
     (stroke (width 0) (type default))
   )
@@
     (stroke (width 0) (type default))
   )
+  (wire (pts (xy 128.27 97.79) (xy 128.27 101.6))
+    (stroke (width 0) (type default))
+  )
   (wire (pts (xy 152.4 91.44) (xy 153.67 91.44))
     (stroke (width 0) (type default))
@@
     (stroke (width 0) (type default))
   )
-  (wire (pts (xy 121.92 116.84) (xy 128.27 116.84))
+  (wire (pts (xy 121.92 129.54) (xy 128.27 129.54))
     (stroke (width 0) (type default))
   )
@@
     (stroke (width 0) (type default))
   )
+  (wire (pts (xy 128.27 114.3) (xy 128.27 121.92))
+    (stroke (width 0) (type default))
+  )
   (wire (pts (xy 146.05 116.84) (xy 146.05 118.11))
     (stroke (width 0) (type default))
@@
     (stroke (width 0) (type default))
   )
-  (wire (pts (xy 118.11 109.22) (xy 114.3 109.22))
+  (wire (pts (xy 118.11 121.92) (xy 114.3 121.92))
     (stroke (width 0) (type default))
   )
@@
     (stroke (width 0) (type default))
   )
-  (wire (pts (xy 128.27 109.22) (xy 125.73 109.22))
+  (wire (pts (xy 128.27 121.92) (xy 125.73 121.92))
     (stroke (width 0) (type default))
   )
@@
       (effects (font (size 1.27 1.27)))
     )
-    (property "Footprint" "BKXXXX:BK1198" (at 130.81 71.12 0)
-      (effects (font (size 1.27 1.27)) hide)
+    (property "Footprint" "BKXXXX:BK1198" (at 130.81 83.82 90)
+      (effects (font (size 1.27 1.27)))
     )
     (property "Datasheet" "" (at 144.78 76.2 0)
@@
     )
   )
-  (symbol (lib_id "Device:C") (at 128.27 113.03 0) (unit 1)
+  (symbol (lib_id "Device:C") (at 128.27 125.73 0) (unit 1)
     (in_bom yes) (on_board yes) (dnp no)
-    (property "Reference" "C7" (at 133.35 110.49 0)
-      (effects (font (size 1.27 1.27)) (justify left))
-    )
-    (property "Value" "22pF" (at 132.08 115.57 0)
-      (effects (font (size 1.27 1.27)) (justify left))
-    )
-    (property "Footprint" "" (at 129.2352 116.84 0)
-      (effects (font (size 1.27 1.27)) hide)
-    )
-    (property "Datasheet" "~" (at 128.27 113.03 0)
+    (property "Reference" "C7" (at 133.35 123.19 0)
+      (effects (font (size 1.27 1.27)) (justify left))
+    )
+    (property "Value" "22pF" (at 132.08 128.27 0)
+      (effects (font (size 1.27 1.27)) (justify left))
+    )
+    (property "Footprint" "" (at 129.2352 129.54 0)
+      (effects (font (size 1.27 1.27)) hide)
+    )
+    (property "Datasheet" "~" (at 128.27 125.73 0)
       (effects (font (size 1.27 1.27)) hide)
     )
@@
     )
   )
-  (symbol (lib_id "Device:Crystal") (at 121.92 109.22 0) (unit 1)
-    (in_bom yes) (on_board yes) (dnp no) (fields_autoplaced)
-    (property "Reference" "Y1" (at 121.92 101.6 0)
-      (effects (font (size 1.27 1.27)))
-    )
-    (property "Value" "32.768kHz" (at 121.92 104.14 0)
-      (effects (font (size 1.27 1.27)))
-    )
-    (property "Footprint" "" (at 121.92 109.22 0)
-      (effects (font (size 1.27 1.27)) hide)
-    )
-    (property "Datasheet" "~" (at 121.92 109.22 0)
+  (symbol (lib_id "Device:R") (at 128.27 105.41 180) (unit 1)
+    (in_bom yes) (on_board yes) (dnp no)
+    (property "Reference" "R18" (at 125.73 105.41 90)
+      (effects (font (size 1.27 1.27)))
+    )
+    (property "Value" "270K" (at 125.73 100.33 90)
+      (effects (font (size 1.27 1.27)))
+    )
+    (property "Footprint" "" (at 130.048 105.41 90)
+      (effects (font (size 1.27 1.27)) hide)
+    )
+    (property "Datasheet" "~" (at 128.27 105.41 0)
+      (effects (font (size 1.27 1.27)) hide)
+    )
+    (pin "1")
+    (pin "2")
+    (instances
+      (project "Basic_Setup"
+        (path "/cf4feedd-3416-459a-83d0-42e924d6c0b9"
+          (reference "R18") (unit 1)
+        )
+      )
+    )
+  )
+  (symbol (lib_id "Device:Crystal") (at 121.92 121.92 0) (unit 1)
+    (in_bom yes) (on_board yes) (dnp no)
+    (property "Reference" "Y1" (at 121.92 114.3 0)
+      (effects (font (size 1.27 1.27)) hide)
+    )
+    (property "Value" "32.768kHz" (at 121.92 128.27 0)
+      (effects (font (size 1.27 1.27)))
+    )
+    (property "Footprint" "" (at 121.92 121.92 0)
+      (effects (font (size 1.27 1.27)) hide)
+    )
+    (property "Datasheet" "~" (at 121.92 121.92 0)
       (effects (font (size 1.27 1.27)) hide)
     )
@@
         (path "/cf4feedd-3416-459a-83d0-42e924d6c0b9"
           (reference "#PWR014") (unit 1)
+        )
+      )
+    )
+  )
+  (symbol (lib_id "Device:R") (at 121.92 114.3 270) (unit 1)
+    (in_bom yes) (on_board yes) (dnp no)
+    (property "Reference" "R19" (at 121.92 116.84 90)
+      (effects (font (size 1.27 1.27)))
+    )
+    (property "Value" "10M" (at 116.84 116.84 90)
+      (effects (font (size 1.27 1.27)))
+    )
+    (property "Footprint" "" (at 121.92 112.522 90)
+      (effects (font (size 1.27 1.27)) hide)
+    )
+    (property "Datasheet" "~" (at 121.92 114.3 0)
+      (effects (font (size 1.27 1.27)) hide)
+    )
+    (pin "1")
+    (pin "2")
+    (instances
+      (project "Basic_Setup"
+        (path "/cf4feedd-3416-459a-83d0-42e924d6c0b9"
+          (reference "R19") (unit 1)
         )
       )
@@
     )
   )
-  (symbol (lib_id "Device:C") (at 114.3 113.03 0) (unit 1)
+  (symbol (lib_id "Device:C") (at 114.3 125.73 0) (unit 1)
     (in_bom yes) (on_board yes) (dnp no)
-    (property "Reference" "C6" (at 106.68 111.76 0)
-      (effects (font (size 1.27 1.27)) (justify left))
-    )
-    (property "Value" "22pF" (at 106.68 115.57 0)
-      (effects (font (size 1.27 1.27)) (justify left))
-    )
-    (property "Footprint" "" (at 115.2652 116.84 0)
-      (effects (font (size 1.27 1.27)) hide)
-    )
-    (property "Datasheet" "~" (at 114.3 113.03 0)
+    (property "Reference" "C6" (at 106.68 124.46 0)
+      (effects (font (size 1.27 1.27)) (justify left))
+    )
+    (property "Value" "22pF" (at 106.68 128.27 0)
+      (effects (font (size 1.27 1.27)) (justify left))
+    )
+    (property "Footprint" "" (at 115.2652 129.54 0)
+      (effects (font (size 1.27 1.27)) hide)
+    )
+    (property "Datasheet" "~" (at 114.3 125.73 0)
       (effects (font (size 1.27 1.27)) hide)
     )
@@
     )
   )
-  (symbol (lib_id "power:GND") (at 121.92 118.11 0) (unit 1)
-    (in_bom yes) (on_board yes) (dnp no) (fields_autoplaced)
-    (property "Reference" "#PWR010" (at 121.92 124.46 0)
-      (effects (font (size 1.27 1.27)) hide)
-    )
-    (property "Value" "GND" (at 121.92 123.19 0)
-      (effects (font (size 1.27 1.27)))
-    )
-    (property "Footprint" "" (at 121.92 118.11 0)
-      (effects (font (size 1.27 1.27)) hide)
-    )
-    (property "Datasheet" "" (at 121.92 118.11 0)
-      (effects (font (size 1.27 1.27)) hide)
-    )
+  (symbol (lib_id "power:GND") (at 121.92 130.81 0) (unit 1)
+    (in_bom yes) (on_board yes) (dnp no) (fields_autoplaced)
+    (property "Reference" "#PWR010" (at 121.92 137.16 0)
+      (effects (font (size 1.27 1.27)) hide)
+    )
+    (property "Value" "GND" (at 121.92 135.89 0)
+      (effects (font (size 1.27 1.27)))
+    )
+    (property "Footprint" "" (at 121.92 130.81 0)
+      (effects (font (size 1.27 1.27)) hide)
+    )
+    (property "Datasheet" "" (at 121.92 130.81 0)
+      (effects (font (size 1.27 1.27)) hide)
+    )
